File: hardware/kicad/swexai_ctrl/experiment.kicad_sch (KiCad schematic)
At the start: 2 parts

Commit message: hardware: inputs complete
Parts:
- R2: footprint (none) -> Resistor_THT:R_Axial_DIN0204_L3.6mm_D1.6mm_P1.90mm_Vertical
Changed lines of the file:
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@@
 			)
 		)
-		(property "Footprint" ""
+		(property "Footprint" "Resistor_THT:R_Axial_DIN0204_L3.6mm_D1.6mm_P1.90mm_Vertical"
 			(at 97.282 72.39 90)
 			(hide yes)
