File: hardware/kicad/swexai_ctrl/untitled.kicad_sch (KiCad schematic)
At the start: 7 parts

Commit message: hardware: inputs complete
Parts:
- D2: value D_TVS -> SMBJ33CA
- R1: value R -> 4.7k
Changed lines of the file:
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@@
 		(fields_autoplaced yes)
 		(property "Reference" "D2"
-			(at 184.15 99.06 0)
+			(at 180.34 97.7899 90)
 			(show_name no)
 			(do_not_autoplace no)
@@
 					(size 1.27 1.27)
 				)
+				(justify left)
 			)
 		)
-		(property "Value" "D_TVS"
-			(at 181.61 99.06 0)
+		(property "Value" "SMBJ33CA"
+			(at 180.34 100.3299 90)
 			(show_name no)
 			(do_not_autoplace no)
@@
 					(size 1.27 1.27)
 				)
+				(justify left)
 			)
 		)
@@
 			)
 		)
-		(property "Value" "R"
+		(property "Value" "4.7k"
 			(at 201.93 96.5199 0)
 			(show_name no)
