File: hardware/kicad/swexai_ctrl/inputs.kicad_sch (KiCad schematic)
At the start: 0 parts

Commit message: hardware: inputs complete
Parts:
- added C10, C11, C4, C5, C6, C7, C8, C9: 100nf, symbol Device:C
- added D10, D11, D4, D5, D6, D7, D8, D9: 1N4148, Diode_SMD:D_SOD-123, symbol Device:D
- added J2, J3, J4, J5, J6, J7, J8, J9: DIGITAL_INPUT_1, symbol Connector:Conn_01x02_Pin
- added R10, R12, R14, R16, R2, R3, R6, R8: 4.7k 0.5W, Resistor_SMD:R_0805_2012Metric, symbol Device:R
- added R11, R13, R15, R17, R4, R5, R7, R9: 10k, Resistor_SMD:R_0805_2012Metric, symbol Device:R
- added U1, U2, U3, U4, U5, U6, U7, U8: PC817, Package_DIP:DIP-4_W7.62mm, symbol Isolator:PC817
Connections:
- new net: D11.1 (K), R16.2, U8.1
- new net: D6.1 (K), R6.2, U3.1
- new net: D9.1 (K), R12.2, U6.1
- new net: D5.1 (K), R3.2, U2.1
- new net: D10.1 (K), R14.2, U7.1
- new net: D8.1 (K), R10.2, U5.1
- new net: D7.1 (K), R8.2, U4.1
- new net: D4.1 (K), R2.2, U1.1
- new net +3V3: R11.2, R13.2, R15.2, R17.2, R4.2, R5.2, R7.2, R9.2
- new net FIELD_BATTER_LOW: J8.1 (Pin_1), R14.1
- new net FIELD_COVER_SW: J3.1 (Pin_1), R3.1
- new net FIELD_ESTOP_SW: J2.1 (Pin_1), R2.1
- new net FIELD_HOME_RADIAL: J7.1 (Pin_1), R12.1
- new net FIELD_HOME_THETA: J6.1 (Pin_1), R10.1
- new net FIELD_SPARE_DI: J9.1 (Pin_1), R16.1
- new net FIELD_START_BTN: J4.1 (Pin_1), R6.1
- new net FIELD_STOP_BTN: J5.1 (Pin_1), R8.1
- new net GND_FIELD: D10.2 (A), D11.2 (A), D4.2 (A), D5.2 (A), D6.2 (A), D7.2 (A), D8.2 (A), D9.2 (A), J2.2 (Pin_2), J3.2 (Pin_2), J4.2 (Pin_2), J5.2 (Pin_2), J6.2 (Pin_2), J7.2 (Pin_2), J8.2 (Pin_2), J9.2 (Pin_2), U1.2, U2.2, U3.2, U4.2, U5.2, U6.2, U7.2, U8.2
- new net GND_LOGIC: C10.2, C11.2, C4.2, C5.2, C6.2, C7.2, C8.2, C9.2, U1.3, U2.3, U3.3, U4.3, U5.3, U6.3, U7.3, U8.3
- new net LOGIC_BATTER_LOW: C10.1, R15.1, U7.4
- new net LOGIC_COVER_SW: C5.1, R5.1, U2.4
- new net LOGIC_ESTOP: C4.1, R4.1, U1.4
- new net LOGIC_HOME_RADIAL: C9.1, R13.1, U6.4
- new net LOGIC_HOME_THETA: C8.1, R11.1, U5.4
- new net LOGIC_SPARE_DI: C11.1, R17.1, U8.4
- new net LOGIC_START_BTN: C6.1, R7.1, U3.4
- new net LOGIC_STOP_BTN: C7.1, R9.1, U4.4

Commit message: hardware: motioncontrol schematics added
Other:
- company: (none) -> SWEXAI AB
- title: (none) -> Inputs
