File: hardware/kicad/swexai_ctrl/outputs.kicad_sch (KiCad schematic)
At the start: 0 parts

Commit message: hardware: motioncontrol schematics added
Parts:
- added J10: FIELD_OUTPUTS_A, symbol Connector:Screw_Terminal_01x04
- added J11: FIELD_OUTPUTS_B, symbol Connector:Screw_Terminal_01x04
- added R18, R19, R20, R21, R22, R23, R24, R25: 1k, symbol Device:R
- added U9: ULN2803A, symbol Transistor_Array:ULN2803A
Connections:
- new net: R21.1, U9.4 (I4)
- new net: R18.1, U9.1 (I1)
- new net: R20.1, U9.3 (I3)
- new net: R22.1, U9.5 (I5)
- new net: R24.1, U9.7 (I7)
- new net: R23.1, U9.6 (I6)
- new net: R19.1, U9.2 (I2)
- new net: R25.1, U9.8 (I8)
- new net +24V_PROTECTED: U9.10 (COM)
- new net FIELD_BUZZER: J10.3 (Pin_3), U9.16 (O3)
- new net FIELD_GREEN_LAMP: J10.1 (Pin_1), U9.18 (O1)
- new net FIELD_HEATER_EN: J10.4 (Pin_4), U9.15 (O4)
- new net FIELD_RADIAL_EN: J11.2 (Pin_2), U9.13 (O6)
- new net FIELD_RED_LAMP: J10.2 (Pin_2), U9.17 (O2)
- new net FIELD_SPARE1: J11.3 (Pin_3), U9.12 (O7)
- new net FIELD_SPARE2: J11.4 (Pin_4), U9.11 (O8)
- new net FIELD_THETA_EN: J11.1 (Pin_1), U9.14 (O5)
- new net GND_FIELD: U9.9 (GND)
- new net LOGIC_BUZZER: R20.2
- new net LOGIC_GREEN_LED: R18.2
- new net LOGIC_HEATER_EN: R21.2
- new net LOGIC_RED_LED: R19.2
- new net LOGIC_SPARE1: R22.2
- new net LOGIC_SPARE2: R23.2
- new net LOGIC_SPARE3: R24.2
- new net LOGIC_SPARE4: R25.2
