File: hardware/kicad/swexai_ctrl/power.kicad_sch (KiCad schematic)
At the start: 7 parts

Commit message: hardware: motioncontrol schematics added
Parts:
- added J_5V_INPUT1: 5V_CONTROL_INPUT, symbol Connector_Generic:Conn_01x02
Connections:
- net GND renamed GND_LOGIC
- net GND_LOGIC: now also J_5V_INPUT1.2 (Pin_2)
- new net +5V_CONTROL: J_5V_INPUT1.1 (Pin_1)
