File: hardware/kicad/swexai_ctrl/swexai_ctrl.kicad_sch (KiCad schematic)
At the start: 0 parts

Commit message: hardware: complete Power.sch with input protection and footprints
Other:
- added sheet Connector (connector.kicad_sch)
- added sheet Experiment (experiment.kicad_sch)
- added sheet Inputs (inputs.kicad_sch)
- added sheet Outputs (outputs.kicad_sch)
- added sheet Power (untitled.kicad_sch)
- added sheet STM32_Interface (stm32_interface.kicad_sch)
- added sheet Stepper (stepper.kicad_sch)
- added sheet Temperature (temperature.kicad_sch)

Commit message: hardware: inputs complete
Other:
- removed sheet Experiment
Changed lines of the file:
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@@
-	)
-	(sheet
-		(at 1121.41 824.23)
-		(size 466.09 240.03)
-		(exclude_from_sim no)
-		(in_bom yes)
-		(on_board yes)
-		(dnp no)
-		(fields_autoplaced yes)
-		(stroke
-			(width 0.1524)
-			(type solid)
-		)
-		(fill
-			(color 0 0 0 0)
-		)
-		(property "Sheetname" "Experiment"
-			(at 1121.41 823.5184 0)
-			(show_name no)
-			(do_not_autoplace no)
-			(effects
-				(font
-					(size 1.27 1.27)
-				)
-				(justify left bottom)
-			)
-		)
-		(property "Sheetfile" "experiment.kicad_sch"
-			(at 1121.41 1064.8446 0)
-			(show_name no)
-			(do_not_autoplace no)
-			(effects
-				(font
-					(size 1.27 1.27)
-				)
-				(justify left top)
-			)
-		)
-		(instances
-			(project "swexai_ctrl"
-				(path "/e84fb207-b24a-4674-962a-61fd98366889"
-					(page "9")
-				)
-			)
-		)
 	)
 	(sheet

Commit message: hardware: motioncontrol schematics added
Other:
- sheet Inputs renamed DigitalInputs
- sheet Outputs renamed DigitalOutputs
- sheet Stepper renamed MotionControl
- removed sheet Connector
- sheet MotionControl: file stepper.kicad_sch -> motioncontrol.kicad_sch
- sheet Power: file untitled.kicad_sch -> power.kicad_sch
Changed lines of the file:
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@@
 			(color 0 0 0 0)
 		)
-		(property "Sheetname" "Outputs"
+		(property "Sheetname" "DigitalOutputs"
 			(at 471.17 18.3384 0)
 			(show_name no)
@@
 	)
 	(sheet
-		(at 1154.43 443.23)
-		(size 490.22 254)
-		(exclude_from_sim no)
-		(in_bom yes)
-		(on_board yes)
-		(dnp no)
-		(fields_autoplaced yes)
-		(stroke
-			(width 0.1524)
-			(type solid)
-		)
-		(fill
-			(color 0 0 0 0)
-		)
-		(property "Sheetname" "Connector"
-			(at 1154.43 442.5184 0)
-			(show_name no)
-			(do_not_autoplace no)
-			(effects
-				(font
-					(size 1.27 1.27)
-				)
-				(justify left bottom)
-			)
-		)
-		(property "Sheetfile" "connector.kicad_sch"
-			(at 1154.43 697.8146 0)
-			(show_name no)
-			(do_not_autoplace no)
-			(effects
-				(font
-					(size 1.27 1.27)
-				)
-				(justify left top)
-			)
-		)
-		(instances
-			(project "swexai_ctrl"
-				(path "/e84fb207-b24a-4674-962a-61fd98366889"
-					(page "8")
-				)
-			)
-		)
-	)
-	(sheet
 		(at 433.07 339.09)
 		(size 410.21 264.16)
@@
 			(color 0 0 0 0)
 		)
-		(property "Sheetname" "Stepper"
+		(property "Sheetname" "MotionControl"
 			(at 433.07 338.3784 0)
 			(show_name no)
@@
 			)
 		)
-		(property "Sheetfile" "stepper.kicad_sch"
+		(property "Sheetfile" "motioncontrol.kicad_sch"
 			(at 433.07 603.8346 0)
 			(show_name no)
@@
 			(color 0 0 0 0)
 		)
-		(property "Sheetname" "Inputs"
+		(property "Sheetname" "DigitalInputs"
 			(at 2.54 668.5784 0)
 			(show_name no)
@@
 			)
 		)
-		(property "Sheetfile" "untitled.kicad_sch"
+		(property "Sheetfile" "power.kicad_sch"
 			(at 5.08 591.1346 0)
 			(show_name no)
