File: hardware/kicad/swexai_ctrl/temperature.kicad_sch (KiCad schematic)
At the start: 0 parts

Commit message: hardware: motioncontrol schematics added
Parts:
- added C1, C2: 100nF, symbol Device:C
- added C3, C4: 10nF, symbol Device:C
- added J1: PT100_3WIRE, symbol Sensor_Temperature:PT100
- added RREF: precision reference resistor, symbol Device:R
- added U11: MAX31865xAP, Package_SO:SSOP-20_5.3x7.2mm_P0.65mm, symbol Sensor_Temperature:MAX31865xAP
Connections:
- new net: U11.13 (GND), U11.19 (GND)
